File: 2-Electrical/0 - Development Drawings/1 - Main Board/5 - CAD project/FRA_Sensor_v1/FRA_Sensor_v1.brd (EAGLE design)
At the start: 79 x 94 mm, 106 parts, among them IC1 CP2101, IC2 LMV611, IC3 TS520533, J1 FTDI, J3 USB, Q1 Si2300DS, T1 BC847, T2 BC847, T3 BC847, U1 DS1307Z, U2 ESP-WROOM-32, Y2 32.768kHz, Y3 32.768kHz

Commit message: sch update
Parts:
- added J2: 2X6 FEMALE, SparkFun-Connectors:2X6
- added J4: (no value), sd-mmc:SDCMF-10915W010
- added R17: 47, resistor:R0603
Connections:
- new net VDD: J4.4
- new net VSS1: J4.3
- new net VSS2: J4.6
- net GND: now also J4.M1, J4.M2, J4.M3, J4.M4
Routing:
- net 3.3V: track 357.0 -> 353.8 mm
Changed lines of the file:
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@@
 <element name="R24" library="resistor" package="R0603" value="100" x="-26.67" y="-217.17"/>
 <element name="U$3" library="adafruit" package="MICROSD" value="MICROSD" x="-43.18" y="-198.12"/>
+<element name="J2" library="SparkFun-Connectors" package="2X6" value="2X6 FEMALE" x="-41.91" y="-224.79">
+<attribute name="PROD_ID" value="CONN-12423" x="-41.91" y="-224.79" size="1.778" layer="27" display="off"/>
+</element>
+<element name="J4" library="sd-mmc" package="SDCMF-10915W010" value="" x="-59.69" y="-203.2"/>
+<element name="R17" library="resistor" package="R0603" value="47" x="-71.12" y="-231.14"/>
 </elements>
 <signals>
@@
 <contactref element="JTAG1" pad="7"/>
 <contactref element="R9" pad="2"/>
+<contactref element="J4" pad="M1"/>
+<contactref element="J4" pad="M2"/>
+<contactref element="J4" pad="M3"/>
+<contactref element="J4" pad="M4"/>
+<wire x1="-47.498" y1="-191.77" x2="-45.72" y2="-205.74" width="0" layer="19" extent="1-1"/>
+<wire x1="-25.82" y1="-196.85" x2="-45.72" y2="-205.74" width="0" layer="19" extent="1-1"/>
 <wire x1="-24.13" y1="-175.95" x2="-25.82" y2="-196.85" width="0" layer="19" extent="1-1"/>
 <wire x1="-4.867865625" y1="-181.030240625" x2="-24.13" y2="-175.95" width="0" layer="19" extent="1-1"/>
@@
 <wire x1="-2.327865625" y1="-181.030240625" x2="-3.597865625" y2="-181.030240625" width="0" layer="19" extent="1-1"/>
 <wire x1="-1.057865625" y1="-181.030240625" x2="-2.327865625" y2="-181.030240625" width="0" layer="19" extent="1-1"/>
+<wire x1="-72.898" y1="-191.77" x2="-47.498" y2="-191.77" width="0" layer="19" extent="1-1"/>
+<wire x1="-72.898" y1="-205.74" x2="-72.898" y2="-191.77" width="0" layer="19" extent="1-1"/>
 <wire x1="-17.088265625" y1="-139.514178125" x2="-24.13" y2="-175.95" width="0" layer="19" extent="1-1"/>
 <wire x1="-17.088265625" y1="-135.3515125" x2="-17.088265625" y2="-139.514178125" width="0" layer="19" extent="1-1"/>
@@
 <contactref element="TP11" pad="TP"/>
 <contactref element="U2" pad="2"/>
-<contactref element="C25" pad="1"/>
-<contactref element="C24" pad="1"/>
 <wire x1="19.3675" y1="23.4175" x2="19.3675" y2="24.13" width="0.6096" layer="16"/>
 <wire x1="19.3675" y1="24.13" x2="18.415" y2="25.0825" width="0.6096" layer="16"/>
@@
 <wire x1="75.93" y1="77.4225" x2="75.8825" y2="77.47" width="0.3048" layer="1"/>
 <wire x1="75.2475" y1="78.105" x2="75.2475" y2="78.8175" width="0.3048" layer="1"/>
-<wire x1="75.2475" y1="78.8175" x2="75.0075" y2="79.0575" width="0.3048" layer="1"/>
-<wire x1="75.0075" y1="81.915" x2="75.0075" y2="79.0575" width="0.3048" layer="1"/>
 <via x="73.025" y="45.085" extent="1-16" drill="0.4" diameter="0.8128"/>
 <wire x1="73.025" y1="45.085" x2="69.85" y2="45.085" width="0.3048" layer="16"/>
@@
 <contactref element="R7" pad="1"/>
 <contactref element="R8" pad="2"/>
+<contactref element="C25" pad="1"/>
+<contactref element="C24" pad="1"/>
 <wire x1="-27.52" y1="-186.69" x2="-25.82" y2="-191.77" width="0" layer="19" extent="1-1"/>
 <wire x1="-18.816465625" y1="-153.483171875" x2="-27.52" y2="-186.69" width="0" layer="19" extent="1-1"/>
@@
 <wire x1="21.2725" y1="56.1975" x2="22.5425" y2="55.5625" width="0" layer="19" extent="16-16"/>
 <wire x1="72.0725" y1="81.915" x2="72.0725" y2="81.915" width="0" layer="19" extent="1-16"/>
+<wire x1="75.0075" y1="81.915" x2="74.93" y2="81.915" width="0" layer="19" extent="1-1"/>
+<wire x1="75.0075" y1="79.0575" x2="75.2475" y2="79.0575" width="0" layer="19" extent="1-1"/>
 <wire x1="20.955" y1="56.515" x2="21.2725" y2="56.1975" width="0" layer="19" extent="16-16"/>
 <wire x1="71.755" y1="81.28" x2="72.0725" y2="81.915" width="0" layer="19" extent="16-16"/>
@@
 <contactref element="U2" pad="30"/>
 </signal>
+<signal name="VSS2">
+<contactref element="J4" pad="6"/>
+</signal>
+<signal name="VSS1">
+<contactref element="J4" pad="3"/>
+</signal>
+<signal name="VDD">
+<contactref element="J4" pad="4"/>
+</signal>
 </signals>

Commit message: sch
Parts:
- added C7, C8: DNI, resistor:C0603K
- added R26: 0, resistor:R0603
- added R27: DNI, resistor:R0603
Connections:
- new net N$9: C7.1, C8.2, R26.2, R27.1, U$1.4
- net 3.3V: now also C8.1, R26.1; no longer U$1.4
- net GND: now also C7.2, R27.2
Routing:
- net 3.3V: track 353.8 -> 353.2 mm
Changed lines of the file:
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@@
 <element name="J4" library="sd-mmc" package="SDCMF-10915W010" value="" x="-59.69" y="-203.2"/>
 <element name="R17" library="resistor" package="R0603" value="47" x="-71.12" y="-231.14"/>
+<element name="R26" library="resistor" package="R0603" value="0" x="-71.12" y="-236.22"/>
+<element name="R27" library="resistor" package="R0603" value="DNI" x="-71.12" y="-241.3"/>
+<element name="C7" library="resistor" package="C0603K" value="DNI" x="-71.12" y="-246.38"/>
+<element name="C8" library="resistor" package="C0603K" value="DNI" x="-71.12" y="-251.46"/>
 </elements>
 <signals>
@@
 <contactref element="J4" pad="M3"/>
 <contactref element="J4" pad="M4"/>
+<contactref element="C7" pad="2"/>
+<contactref element="R27" pad="2"/>
 <wire x1="-47.498" y1="-191.77" x2="-45.72" y2="-205.74" width="0" layer="19" extent="1-1"/>
 <wire x1="-25.82" y1="-196.85" x2="-45.72" y2="-205.74" width="0" layer="19" extent="1-1"/>
@@
 <wire x1="-72.898" y1="-191.77" x2="-47.498" y2="-191.77" width="0" layer="19" extent="1-1"/>
 <wire x1="-72.898" y1="-205.74" x2="-72.898" y2="-191.77" width="0" layer="19" extent="1-1"/>
+<wire x1="-70.27" y1="-241.3" x2="-72.898" y2="-205.74" width="0" layer="19" extent="1-1"/>
+<wire x1="-70.245" y1="-246.38" x2="-70.27" y2="-241.3" width="0" layer="19" extent="1-1"/>
 <wire x1="-17.088265625" y1="-139.514178125" x2="-24.13" y2="-175.95" width="0" layer="19" extent="1-1"/>
 <wire x1="-17.088265625" y1="-135.3515125" x2="-17.088265625" y2="-139.514178125" width="0" layer="19" extent="1-1"/>
@@
 <contactref element="R25" pad="2"/>
 <contactref element="C21" pad="1"/>
-<contactref element="U$1" pad="4"/>
 <contactref element="L1" pad="2"/>
 <contactref element="C23" pad="+"/>
@@
 <wire x1="38.6325" y1="22.5425" x2="38.4175" y2="22.5425" width="0.3048" layer="1"/>
 <wire x1="37.1475" y1="23.8125" x2="37.1475" y2="23.89" width="0.3048" layer="16"/>
-<wire x1="23.7824" y1="41.2775" x2="23.7824" y2="40.64" width="0.8128" layer="16"/>
 <wire x1="23.7824" y1="40.64" x2="23.7824" y2="40.1126" width="0.8128" layer="16"/>
 <wire x1="23.7824" y1="40.1126" x2="24.2075" y2="39.6875" width="0.8128" layer="16"/>
@@
 <contactref element="C25" pad="1"/>
 <contactref element="C24" pad="1"/>
+<contactref element="R26" pad="1"/>
+<contactref element="C8" pad="1"/>
 <wire x1="-27.52" y1="-186.69" x2="-25.82" y2="-191.77" width="0" layer="19" extent="1-1"/>
 <wire x1="-18.816465625" y1="-153.483171875" x2="-27.52" y2="-186.69" width="0" layer="19" extent="1-1"/>
+<wire x1="-71.97" y1="-236.22" x2="-25.82" y2="-191.77" width="0" layer="19" extent="1-1"/>
+<wire x1="-71.995" y1="-251.46" x2="-71.97" y2="-236.22" width="0" layer="19" extent="1-1"/>
 <wire x1="11.43" y1="2.325" x2="-18.816465625" y2="-153.483171875" width="0" layer="19" extent="1-1"/>
 <wire x1="21.2725" y1="56.1975" x2="22.5425" y2="55.5625" width="0" layer="19" extent="16-16"/>
@@
 <contactref element="J4" pad="4"/>
 </signal>
+<signal name="N$9">
+<contactref element="R27" pad="1"/>
+<contactref element="R26" pad="2"/>
+<contactref element="C8" pad="2"/>
+<contactref element="C7" pad="1"/>
+<contactref element="U$1" pad="4"/>
+<wire x1="-71.995" y1="-246.38" x2="-70.245" y2="-251.46" width="0" layer="19" extent="1-1"/>
+<wire x1="-71.97" y1="-241.3" x2="-71.995" y2="-246.38" width="0" layer="19" extent="1-1"/>
+<wire x1="-70.27" y1="-236.22" x2="-71.97" y2="-241.3" width="0" layer="19" extent="1-1"/>
+<wire x1="23.7824" y1="41.2775" x2="-70.27" y2="-236.22" width="0" layer="19" extent="1-16"/>
+</signal>
 </signals>

Commit message: power circuits
Parts:
- removed BT1: 3V, SparkFun-Batteries:BATTCOM_20MM_PTH_KIT
- removed C26, C28: 100n, resistor:C0603K
- removed C27: 10u, resistor:C0603K
- removed TP7: TPTP10R, testpad:TP10R
- removed U$1: LM3671, texas-custom:SOT23-5
- removed U1: DS1307Z, SparkFun-Clocks:SO08-0.15
- removed Y2: 32.768kHz, SparkFun-Clocks:CRYSTAL-SMD-3.2X1.5MM
- added C11: 10u, resistor:C0603K
- added C12: 100n, resistor:C0603K
- added L2: TYS60451R5N-10 1.5uH, FRA_eagle_lib:VLS3012HBX-1R5M
- added Q2, Q3: (no value), microbuilder:SOT23-WIDE
- added R28: 10k, resistor:R0603
- added R29: DNI, resistor:R0603
- added R30: 45.3k, resistor:R0603
- added U$4, U$5: TPS5632149DDCR, FRA_eagle_lib:SOT23-6
- C10: value 100n -> 10u
- C9: value 10u -> 100n
- R16: value 12k -> 0
- R22: value 0 -> 10k
- moved C6 382.1 mm to (-71.1, -276.9), flipped to the top, turned to 0 degrees
- moved C9 370.2 mm to (-71.1, -281.9), flipped to the top, turned to 0 degrees
- moved R22 358.8 mm to (-71.1, -302.3), flipped to the top, turned to 0 degrees
- moved C1 328.6 mm to (-71.1, -266.7), flipped to the top
- moved C10 322.5 mm to (-71.1, -287.0), flipped to the top, turned to 0 degrees
- moved R16 312.5 mm to (-71.1, -271.8), flipped to the top, turned to 0 degrees
- moved U$3 25.0 mm to (-67.3, -191.8)
- moved JTAG1 4.02 mm to (-7.41, -180.5)
- moved J2 1.27 mm to (-43.2, -224.8)
Connections:
- removed net N$30: U1.1, Y2.P$2
- removed net N$31: U1.2, Y2.P$1
- removed net SPI_HOLD: TP7.TP
- removed net SQW: R16.1, U1.7
- removed net VBAT: BT1.1, U1.3
- new net N$15: R16.2, U$4.6
- new net N$23: R22.1, U$4.5
- new net N$24: R28.1, R29.1, R30.1, U$4.4
- new net VIN: C6.1, C9.1, R22.2, U$4.3
- net 3.3V: now also C11.1, C12.1, L2.P$2, R29.2, R30.2; no longer C27.1, C28.1, R16.2, U1.8
- net 5V: no longer C6.1, C9.1, R22.2, U$1.1
- net GND: now also C11.2, C12.2, R28.2, U$4.1; no longer BT1.2, C1.1, C26.2, C27.2, C28.2, U$1.2, U1.4
- net N$16: no longer R22.1
- net N$19: now also C1.2, L2.P$1, U$4.2; no longer C26.1
- net N$27: no longer U$1.3
- net N$3: now also C1.1, R16.1; no longer C1.2, D3.3
- net N$37: no longer U$1.5
- net N$9: no longer U$1.4
- net SCL: no longer U1.6
- net SDA: no longer U1.5
Routing:
- net SDA: track 123.7 -> 0.00 mm, vias 4 -> 0
- net SCL: track 113.2 -> 0.00 mm, vias 4 -> 0
- net GND: track 571.7 -> 492.7 mm, vias 31 -> 29
- net 3.3V: track 353.2 -> 308.8 mm, vias 27 -> 26
- net SPI_HOLD: track 20.9 -> 0.00 mm, vias 2 -> 0
- net 5V: track 194.0 -> 183.5 mm
- net VBAT: track 6.66 -> 0.00 mm
- net N$3: track 3.90 -> 0.00 mm
- net N$30: track 3.60 -> 0.00 mm
- net SQW: track 3.00 -> 0.00 mm
- net N$31: track 2.92 -> 0.00 mm
- net N$37: track 3.33 -> 0.64 mm
- net N$16: track 5.88 -> 5.14 mm

Commit message: sch
Parts:
- added R31, R32, R47, R48: 47, resistor:R0603
Connections:
- net SCL: now also R47.1
- net SDA: now also R32.1
- net VSPI_CS_ETH: now also R48.1
- net VSPI_MISO: now also R31.1
- net VSPI_MOSI: now also R17.1
Changed lines of the file:
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@@
 <element name="Q2" library="microbuilder" package="SOT23-WIDE" value="" x="-71.12" y="-330.2"/>
 <element name="Q3" library="microbuilder" package="SOT23-WIDE" value="" x="-71.12" y="-334.01"/>
+<element name="R31" library="resistor" package="R0603" value="47" x="-71.12" y="-339.09"/>
+<element name="R32" library="resistor" package="R0603" value="47" x="-71.12" y="-344.17"/>
+<element name="R47" library="resistor" package="R0603" value="47" x="-71.12" y="-349.25"/>
+<element name="R48" library="resistor" package="R0603" value="47" x="-71.12" y="-354.33"/>
 </elements>
 <signals>
@@
 <signal name="SCL">
 <contactref element="U2" pad="36"/>
+<contactref element="R47" pad="1"/>
+<wire x1="74.66" y1="58.31" x2="-71.97" y2="-349.25" width="0" layer="19" extent="1-1"/>
 </signal>
 <signal name="SDA">
 <contactref element="U2" pad="33"/>
+<contactref element="R32" pad="1"/>
+<wire x1="70.85" y1="58.31" x2="-71.97" y2="-344.17" width="0" layer="19" extent="1-1"/>
 </signal>
 <signal name="ADC">
@@
 <signal name="VSPI_CS_ETH">
 <contactref element="U2" pad="37"/>
+<contactref element="R48" pad="1"/>
+<wire x1="75.93" y1="58.31" x2="-71.97" y2="-354.33" width="0" layer="19" extent="1-1"/>
 </signal>
 <signal name="VSPI_MISO">
 <contactref element="U2" pad="31"/>
+<contactref element="R31" pad="1"/>
+<wire x1="68.31" y1="58.31" x2="-71.97" y2="-339.09" width="0" layer="19" extent="1-1"/>
 </signal>
 <signal name="VSPI_MOSI">
 <contactref element="U2" pad="30"/>
+<contactref element="R17" pad="1"/>
+<wire x1="-71.97" y1="-231.14" x2="67.04" y2="58.31" width="0" layer="19" extent="1-1"/>
 </signal>
 <signal name="VSS2">

Commit message: SD card connected
Parts:
- removed J1: FTDI, SparkFun-Connectors:1X06_LONGPADS
- removed Q3: (no value), microbuilder:SOT23-WIDE
- removed U$5: TPS5632149DDCR, FRA_eagle_lib:SOT23-6
- added C13, C15, C27, C28, C37, C38, C40: 100n, resistor:C0603K
- added C14, C17, C26, C39: 10u, resistor:C0603K
- added L3: TYS60451R5N-10 1.5uH, FRA_eagle_lib:VLS3012HBX-1R5M
- added R49, R50, R53, R54: 10k, resistor:R0603
- added R51: DNI, resistor:R0603
- added R52: 73.2k, resistor:R0603
- added R55, R63, R66: 47, resistor:R0603
- added R64, R67: 10K, resistor:R0603
- added R65: 0, resistor:R0603
- added U$1: TPS5632149DDCR, FRA_eagle_lib:SOT23-6
- J2: value 2X6 FEMALE -> ETH_CONN
- Q2: value (none) -> FDN306P
- R11: value 12k -> 0
- R25: value 12k -> 10K
- moved R11 407.2 mm to (-71.1, -367.0), turned to 0 degrees
- moved R17 186.7 mm to (-71.1, -417.8)
Connections:
- net N$18 renamed TDICONN
- net N$4 renamed TDOCONN
- net N$5 renamed TMSCONN
- net N$6 renamed VDDPROG
- net N$7 renamed TCKCONN
- net N$8 renamed VCCJTAG
- removed net VSS1: J4.3
- removed net VSS2: J4.6
- new net ADC_CS: R66.2
- new net ADC_CS_MCU: R66.1, U2.11
- new net ETH_CS: R48.2
- new net MISO: J4.7, R31.2, U$3.7
- new net MOSI: J4.2, R17.2, U$3.3
- new net N$20: R11.2, U$1.6
- new net N$21: C13.2, L3.P$1, U$1.2
- new net N$22: R49.1, U$1.5
- new net N$25: R50.1, R51.1, R52.1, U$1.4
- new net N$30: Q2.1, R53.1, R54.2
- new net SCLK: R55.2
- new net SCL_MCU: R47.1, U2.36
- new net SDA_MCU: R32.1, U2.33
- new net SD_CD: J4.10, R64.1, U$3.CD1, U$3.CD2
- new net SD_CS: J4.1, R63.2, U$3.2
- new net SD_CS_MCU: R63.1, U2.10
- new net SENSOR_DET1: C37.1, R67.1, U2.4
- new net VIN_PROTECTED: C14.1, C15.1, C6.1, C9.1, Q2.3, U$1.3, U$4.3
- net 3.3V: now also R64.2, R65.2, R67.2; no longer R11.2
- net 5V: now also C17.1, C26.1, C27.1, L3.P$2, R51.2, R52.2
- net D_N: now also D1.3
- net D_P: now also D2.3
- net GND: now also C14.2, C15.2, C17.2, C26.2, C27.2, C28.2, C37.2, C38.2, C39.2, C40.2, D1.2, D2.2, J4.3, J4.6, R50.2, R53.2, U$1.1, U$3.6, U$3.MT1, U$3.MT2; no longer J1.6
- net N$11: now also C13.1; no longer J1.4
- net RXD0: no longer J1.3
- net SCL: now also R47.2; no longer R47.1, U2.36
- net SDA: now also R32.2; no longer R32.1, U2.33
- net TXD0: no longer J1.2
- net VDD: now also C38.1, R65.1, U$3.4
- net VIN: now also C28.1, Q2.2, R49.2, R54.1; no longer C6.1, C9.1, U$4.3
- net VSPI_SCK: now also R55.1
- net V_USB: now also D1.1, D2.1
Routing:
- net GND: track 492.7 -> 469.8 mm
- net N$11: track 9.78 -> 0.00 mm, vias 1 -> 0
- net TXD0: track 118.2 -> 111.6 mm
- net RXD0: track 122.0 -> 117.5 mm
- net 3.3V: track 308.8 -> 306.9 mm
