File: 2-Electrical/0 - Development Drawings/1 - Main Board/5 - CAD project/FRA_Sensor_v1/FRA_Sensor_v1.brd (EAGLE design)
At the start: 100 x 100 mm, 151 parts, among them IC1 CP2101, IC2 LMV611, IC3 TS520533, J2 ETH_CONN, J3 USB, Q1 Si2300DS, Q2 FDN306P, T1 BC847, T2 BC847, T3 BC847, U2 ESP-WROOM-32, X1 TB001-500-02BE, Y3 32.768kHz

Commit message: digital sensors interface
Parts:
- added C23, C31: 100n, resistor:C0603K
- added J5: WM9734TR-ND, SparkFun-Connectors:USB-B-MICRO-SMD_VERT
- added R26, R27: 10, resistor:R0603
- SENSOR_D1, SENSOR_D2: value SENS1 -> + G SCL SDA
- moved R14 698.5 mm to (-135.9, 165.1)
- moved R15 698.5 mm to (-135.9, 160.0)
- moved R18 698.5 mm to (-135.9, 154.9)
- moved R19 698.5 mm to (-135.9, 149.9)
- moved D6 680.7 mm to (-120.7, 153.7)
- moved C7 651.6 mm to (-127.0, 165.1)
- moved D4 651.6 mm to (-128.3, 139.7)
- moved LIGHT_DR1 651.6 mm to (-118.1, 162.6)
- moved TP1 651.6 mm to (-129.5, 156.2)
- moved TP2 651.6 mm to (-129.5, 152.4)
- moved TP4 651.6 mm to (-129.5, 144.8)
- moved R69 615.4 mm to (-120.7, 146.1)
- moved TP3 613.6 mm to (-106.7, 110.5)
- moved U$5 607.8 mm to (-105.4, 133.3)
- moved U$6 607.8 mm to (-110.5, 133.3)
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- renumbered SENSOR_10 to SENSOR_D2, SENSOR_9 to SENSOR_D1
Connections:
- new net N$4: C23.1, R27.2, SENSOR_D1.1
- new net N$5: C31.1, R26.2, SENSOR_D2.1
- net 3.3V: now also R26.1, R27.1
- net D_N: now also J5.D-
- net D_P: now also J5.D+
- net GND: now also C23.2, C31.2, J5.GND, SENSOR_D1.2, SENSOR_D2.2
- net SCL: now also SENSOR_D1.3, SENSOR_D2.3
- net SDA: now also SENSOR_D1.4, SENSOR_D2.4
- net V_USB: now also J5.VBUS
Routing:
- net DTR: track 40.8 -> 6.98 mm, vias 3 -> 1
- net RTS: track 36.0 -> 2.44 mm, vias 4 -> 0
- net 3.3V: track 29.1 -> 8.92 mm, vias 3 -> 2
- net D_N_CP: track 15.5 -> 4.67 mm, vias 1 -> 0
- net D_P: track 4.76 -> 0.02 mm, vias 1 -> 0
- net D_N: track 4.06 -> 0.08 mm, vias 1 -> 0
- net D_P_CP: track 7.76 -> 5.76 mm, vias 1 -> 0
- net GND: vias 7 -> 2
- removed copper zone on layer 1, net GND
- removed copper zone on layer 16, net GND
Other:
- board text removed: "*"
- board text removed: "+5V"
- board text removed: "U1"
- board text removed: "U4"
- board text removed: "U6"

Commit message: sch
Parts:
- removed C37: 100n, resistor:C0603K
- removed J3: USB, SparkFun-Connectors:USB-MICROB-PTH-MILL
- removed R67: 10K, resistor:R0603
- removed U$3: MICROSD, adafruit:MICROSD
- added C8: 10u, resistor:C0603K
- added FAN_5V: FAN, pinhead:1X02
- added IC4, IC5, IC6: ADS1115BQDGSRQ1, SamacSys_Parts:SOP50P490X110-10N
- added J8: 1140084168, SamacSys_Parts:1140084168
- added JP1: (no value), pinhead:1X05
- added JP2: (no value), pinhead:1X06
- added Q3: Si2300DS, adafruit:SOT23
- added R20: 47, resistor:R0603
- added R41: 0(DNI), resistor:R0603
- added R45: 0, resistor:R0603
- added TP5: TPTP10R, testpad:TP10R
- R21: value 0 -> 1M
- moved R26 240.5 mm to (78.7, 53.3), turned to 90 degrees
- moved C31 235.4 mm to (76.2, 57.8), turned to 90 degrees
- moved R27 233.9 mm to (68.6, 53.3), turned to 90 degrees
- moved C23 232.9 mm to (71.1, 57.8), turned to 90 degrees
- moved C39 208.7 mm to (61.0, 22.2), turned to 180 degrees
- moved R31 206.1 mm to (29.2, 22.9)
- moved R48 205.7 mm to (58.4, 33.0)
- moved C40 205.0 mm to (62.2, 25.4), turned to 90 degrees
- moved R65 198.9 mm to (33.7, 25.4)
- moved C38 193.6 mm to (34.3, 23.5)
- moved R32 192.0 mm to (61.0, 66.7)
- moved R47 192.0 mm to (61.0, 61.6)
- moved R64 181.8 mm to (40.0, 26.7)
- moved D6 132.2 mm to (-52.1, 40.6), turned to 90 degrees
- moved R21 128.4 mm to (-135.9, -78.1), turned to 0 degrees
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Connections:
- removed net SENSOR_DET1: C37.1, R67.1, U2.4
- removed net SHIELD: J3.SHIELD, J3.SHIELD10, J3.SHIELD2, J3.SHIELD3, J3.SHIELD4, J3.SHIELD5, J3.SHIELD6, J3.SHIELD7, J3.SHIELD8, J3.SHIELD9, R21.1
- removed net VDD: C38.1, J4.4, R65.1, U$3.4
- new net FAN: Q3.1, R20.2, R21.1, TP5.TP
- new net FAN_MCU: R20.1, U2.10
- new net N$10: C38.1, J4.4, R65.1
- new net N$8: FAN_5V.1, Q3.3
- new net N$9: D7.K, R41.1, R45.2
- net 3.3V: now also R18.2, R19.2; no longer R67.2
- net 5V: now also C8.1, FAN_5V.2
- net D_N: no longer J3.D-
- net D_P: no longer J3.D+
- net ETH_CS: now also J2.3
- net ETH_INT: now also U2.24
- net ETH_RST: now also U2.26
- net GND: now also C8.2, Q3.2, R45.1; no longer C37.2, D7.K, D8.K, J3.GND, U$3.6, U$3.MT1, U$3.MT2
- net GPIO0: now also R41.2
- net LED: now also D8.K; no longer R18.2, R19.2
- net MISO: now also J2.8; no longer U$3.7
- net MOSI: now also J2.5; no longer U$3.3
- net SCLK: now also J2.6, J4.5
- net SD_CD: no longer U$3.CD1, U$3.CD2
- net SD_CS: no longer U$3.2
- net V_USB: no longer J3.VBUS
Routing:
- net GND: track 26.3 -> 46.6 mm
- net SHIELD: track 2.86 -> 0.00 mm, vias 4 -> 0
- removed copper zone on layer 16, net SHIELD

Commit message: sch and layiout
Parts:
- added C21: 10u, resistor:C0603K
- added FB1, FB2: (no value), microbuilder:0603
- added Q4: Si2300DS, adafruit:SOT23
- moved D1 163.8 mm to (80.5, 8.80), turned to 270 degrees
- moved D2 163.5 mm to (88.0, 10.3), turned to 90 degrees
- moved R2 157.2 mm to (144.5, 11.7), turned to 270 degrees
- moved T2 155.3 mm to (141.0, 9.84), turned to 90 degrees
- moved R1 154.9 mm to (145.1, 14.9), turned to 180 degrees
- moved T1 151.7 mm to (141.0, 13.7), turned to 90 degrees
- moved R44 133.5 mm to (105.7, 21.9), turned to 270 degrees
- moved R42 114.8 mm to (86.4, 13.7), turned to 0 degrees
- moved R43 114.2 mm to (89.4, 14.0), turned to 270 degrees
- moved R40 110.0 mm to (88.3, 21.3), turned to 270 degrees
- moved IC1 107.9 mm to (83.8, 18.1), turned to 90 degrees
- moved R4 102.0 mm to (79.4, 19.4), turned to 270 degrees
- moved R3 100.7 mm to (77.5, 19.4), turned to 270 degrees
- moved X1 90.0 mm to (5.71, 36.8), turned to 270 degrees
- moved U2 83.1 mm to (91.1, 43.8), turned to 0 degrees
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Connections:
- net D_N renamed D_N_
- net D_P renamed D_P_
- new net 5V1: C21.1
- new net SD_VDD: C38.1, J4.4, J8.4, R65.1
- net GND: now also C21.2, J5.P1, J5.P2, J5.P3, J8.6, J8.CD1, Q4.2
- net MISO: now also J8.7
- net MOSI: now also J8.3
- net N$10: now also Q4.3; no longer C38.1, J4.4, R65.1
- net SCLK: now also J8.5
- net SD_CD: now also J8.CD2
- net SD_CS: now also J8.2
Routing:
- net V_USB: track 0.00 -> 24.1 mm, vias 0 -> 3
- net GND: track 46.6 -> 26.3 mm
- net D_P_: track 0.00 -> 6.90 mm
- net D_N_: track 0.00 -> 5.92 mm
- net 3.3V: track 8.92 -> 4.75 mm, vias 2 -> 0
- net RXD0_CP2101IN: track 5.87 -> 4.23 mm
- net TXD0_CP2101: track 3.39 -> 2.12 mm
- net N$39: track 5.53 -> 4.37 mm
- net D_P_CP: track 5.76 -> 6.54 mm, vias 0 -> 2

Commit message: jtag layout
Parts:
- removed C4: 10u, resistor:C0603K
- removed DRILEGEND: (no value), drilegend:DRILEGEND
- moved C14 207.1 mm to (92.6, 139.8)
- moved C15 207.1 mm to (99.0, 141.1)
- moved C26 207.1 mm to (107.9, 141.1)
- moved C28 207.1 mm to (124.4, 171.6)
- moved C7 207.1 mm to (78.7, 189.4)
- moved D4 207.1 mm to (77.4, 164.0)
- moved IC3 207.1 mm to (168.3, 181.0)
- moved L3 207.1 mm to (110.4, 146.2)
- moved Q1 207.1 mm to (168.3, 201.9)
- moved R11 207.1 mm to (101.5, 152.5)
- moved R23 207.1 mm to (167.4, 152.7)
- moved R52 207.1 mm to (116.8, 143.6)
- moved R53 207.1 mm to (130.7, 169.0)
- moved R54 207.1 mm to (124.4, 167.8)
- moved R56 207.1 mm to (167.4, 225.7)
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Connections:
- net 5V: no longer C4.1, C5.1
- net GND: no longer C4.2
- net V_USB: now also C5.1
Routing:
- net GND: track 26.3 -> 195.3 mm, vias 2 -> 6
- net NRST: track 0.00 -> 94.8 mm, vias 0 -> 5
- net 3.3V: track 4.75 -> 49.5 mm, vias 0 -> 3
- net RXD0: track 0.00 -> 33.0 mm
- net TXD0: track 0.00 -> 32.9 mm
- net GPIO0: track 0.00 -> 31.5 mm, vias 0 -> 3
- net DTR: track 6.98 -> 37.5 mm, vias 1 -> 2
- net RTS: track 2.44 -> 31.7 mm, vias 0 -> 2
- net TDICONN: track 0.00 -> 11.8 mm, vias 0 -> 2
- net TDOCONN: track 0.00 -> 11.6 mm
- net N$39: track 4.37 -> 14.9 mm
- net VDDPROG: track 0.00 -> 9.15 mm, vias 0 -> 2
- net MTMS: track 0.00 -> 7.45 mm
- net N$38: track 5.39 -> 10.4 mm
- net TMSCONN: track 0.00 -> 4.34 mm
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Other:
- board text removed: "U3"

Commit message: power layouts
Parts:
- removed R66: 47, resistor:R0603
- added FB3, FB4, FB5, FB6: (no value), microbuilder:0603
- added Q5, Q6: Si2300DS, adafruit:SOT23
- added Q7: 100A/100V/6.8mΩ, microbuilder:TO252
- added R46, R67, R70, R71: 10k, resistor:R0603
- added TP6, TP7: TPTP10R, testpad:TP10R
- L2, L3: device FRA_eagle_lib:VLS3012HBX-1R5M -> FRA_eagle_lib:TYS60451R5N-10
- R32, R47: value 47 -> 0
- moved U$4 234.5 mm to (42.3, 10.3), turned to 270 degrees
- moved C6 222.8 mm to (41.0, 3.58)
- moved C1 220.7 mm to (46.1, 13.6), turned to 180 degrees
- moved R16 217.7 mm to (46.1, 11.9), turned to 180 degrees
- moved C9 216.7 mm to (41.0, 5.35)
- moved R49 211.1 mm to (19.4, 3.49)
- moved C10 204.5 mm to (39.8, 14.7)
- moved TP11 202.5 mm to (21.9, 35.6)
- moved R22 201.9 mm to (37.8, 3.58)
- moved C11 198.7 mm to (39.8, 16.3)
- moved C12 192.9 mm to (39.8, 17.9)
- moved R28 188.5 mm to (46.6, 8.88)
- moved R29 186.0 mm to (46.6, 6.76)
- moved R30 183.4 mm to (46.6, 4.64)
- moved TP1 181.5 mm to (35.4, 3.60)
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Connections:
- removed net 5V1: C21.1
- removed net ADC_CS: R66.2
- removed net ADC_CS_MCU: R66.1, U2.11
- removed net N$30: Q2.1, R53.1, R54.2
- new net GNDIN: FB5.1, FB6.1, J1.1, J1.2, X1.2
- new net SCL_5V: Q6.3, R71.2
- new net SDA_5V: Q5.3, R67.2
- new net VGI: Q2.1, Q7.1, R53.1, R54.2
- new net VIN_IN: FB3.1, FB4.1, J1.3, X1.1
- net 3.3V: now also Q5.1, Q6.1, R46.1, R70.1
- net 5V: now also R67.1, R71.1
- net GND: now also FB5.2, FB6.2; no longer J1.1, J1.2, X1.2
- net SCL: now also Q6.2, R70.2, TP7.TP
- net SDA: now also Q5.2, R46.2, TP6.TP
- net VIN: now also FB3.2, FB4.2, Q2.3, Q7.3; no longer J1.3, Q2.2, R22.2, R49.2, X1.1
- net VIN_PROTECTED: now also Q2.2, Q7.2, R22.2, R49.2; no longer Q2.3
Routing:
- net GND: track 195.3 -> 334.4 mm, vias 6 -> 28
- net VIN_PROTECTED: track 0.00 -> 41.4 mm
- net 5V: track 0.00 -> 33.4 mm
- net VGI: track 0.00 -> 25.8 mm, vias 0 -> 2
- net 3.3V: track 49.5 -> 73.8 mm
- net VIN: track 0.00 -> 19.2 mm
- net N$22: track 0.00 -> 16.6 mm, vias 0 -> 2
- net N$23: track 0.00 -> 15.2 mm, vias 0 -> 2
- net N$21: track 0.00 -> 13.5 mm, vias 0 -> 2
- net N$19: track 0.00 -> 13.2 mm, vias 0 -> 2
- net N$25: track 0.00 -> 7.50 mm
- net N$24: track 0.00 -> 6.64 mm
- net GNDIN: track 0.00 -> 4.00 mm, vias 0 -> 5
- net N$20: track 0.00 -> 2.21 mm
- net N$11: track 0.00 -> 1.97 mm
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- added copper zone on layer 1, net 3.3V
- added copper zone on layer 1, net 5V
- added copper zone on layer 1, net GND
- added copper zone on layer 16, net GND
- added copper zone on layer 1, net GNDIN
- added copper zone on layer 16, net GNDIN
- added copper zone on layer 1, net VIN
- added copper zone on layer 1, net VIN_IN
- added copper zone on layer 16, net VIN_IN
- added copper zone on layer 1, net VIN_PROTECTED
Other:
- board text added: "5V"
