File: 2-Electrical/0 - Development Drawings/1 - Main Board/5 - CAD project/FRA_Sensor_v1/FRA_Sensor_v1.brd (EAGLE design)
At the start: 100 x 100 mm, 237 parts, among them IC1 CP2101, IC2 LMV611, IC3 TS520533, IC4 ADS1115BQDGSRQ1, IC5 ADS1115BQDGSRQ1, IC7 LMP91000SD_NOPB, IC8 PCA9555PW, IC9 LDK320ADU50R, J2 ETH_CONN, J5 WM9734TR-ND, J8 1140084168, Q1 Si2300DS, Q10 FDN306P, Q11 FDN306P, Q12 FDN306P, Q13 FDN306P, Q14 FDN306P, Q15 FDN306P, Q16 FDN306P, Q17 FDN306P, Q2 FDN306P, Q3 Si2300DS, Q5 FDN306P, Q6 FDN306P, Q7 100A/100V/6.8mΩ, Q8 FDN306P, Q9 FDN306P, T1 BC847, T2 BC847, T3 BC847, U1 PCA9509DP, U2 ESP-WROOM-32, X1 TB001-500-02BE, Y3 32.768kHz

Commit message: sch update layout update
Parts:
- removed C20, C22: 10u, resistor:C0603K
- removed C32, C33, C34: 100n, resistor:C0603K
- removed C35, C36: 1u, resistor:C0603K
- removed D3: BAS17, nxp_60:SOT23
- removed IC3: TS520533, v-reg:SOT25
- removed IC7: LMP91000SD_NOPB, SamacSys_Parts:SON50P400X400X80-15N
- removed Q1: Si2300DS, adafruit:SOT23
- removed Q16, Q17: FDN306P, microbuilder:SOT23-WIDE
- removed R33, R66, R79, R80: 10k, resistor:R0603
- removed R34, R35, R36: 47k, resistor:R0603
- removed R37: 27k, resistor:R0603
- removed R38: 0, resistor:R0603
- removed R39: 12k, resistor:R0603
- removed R56: 5.1k, resistor:R0603
- removed R57: 0R, resistor:R0603
- removed R58, R60, R61, R62: (DNI), resistor:R0603
- removed R59: 1M, resistor:R0603
- removed S$1: CITIPEL_4P50, FRA_eagle_lib:TH3_4P50
- removed S$2: FIGARO_2611, FRA_eagle_lib:TH4_TGS2611
- removed T3: BC847, nxp_60:SOT23
- removed T4: (no value), transistor-neu-to92:SOT223
- removed TP18: TPTP10R, testpad:TP10R
- removed U$17, U$18: CONN_03X2_WE_61200621621, FRA_eagle_lib:WE_61200621621
- added R14: 0(DNI), resistor:R0603
- added R15, R18: 10k, resistor:R0603
- added SENSOR_D3: + G SCL SDA, pinhead:1X04
- added TP21: TPTP10R, testpad:TP10R
- C18: value 1n -> 100n
- C19: value 10u -> 100n
- C37, C41: value 1u -> 10u
- C4: value 1u -> 100n
- IC2: value LMV611 -> ADS1115BQDGSRQ1; device linear:SC70-5L -> SamacSys_Parts:SOP50P490X110-10N
- R42: value 2k(NC) -> 10k
- R81, R82: value 10k -> 2k2
- moved IC2 159.3 mm to (56.6, 65.0), flipped to the top, turned to 180 degrees
- moved C4 159.0 mm to (56.6, 62.2), flipped to the top
- moved C19 155.8 mm to (55.7, 69.4), flipped to the top, turned to 90 degrees
- moved C18 150.1 mm to (60.1, 69.4), flipped to the top
- moved U$16 91.5 mm to (50.0, 77.0), turned to 270 degrees
- moved U$15 85.5 mm to (50.0, 90.0), turned to 270 degrees
- moved R77 83.1 mm to (45.1, 65.7), turned to 180 degrees
- moved R78 83.1 mm to (49.8, 65.7), turned to 180 degrees
- moved Q14 76.0 mm to (45.1, 69.4)
- moved Q15 75.1 mm to (49.8, 69.4)
- moved TP12 70.6 mm to (84.0, 65.3)
- moved R81 67.4 mm to (46.4, 49.8), turned to 0 degrees
- moved R82 66.6 mm to (49.8, 49.8), turned to 180 degrees
- moved IC4 60.5 mm to (79.7, 65.2), turned to 180 degrees
- moved C44 58.8 mm to (79.7, 62.5)
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Connections:
- removed net 3V3_TGS2611: C36.1, IC3.5, R61.2
- removed net AA1: R66.1
- removed net ADC3_3: U$17.2
- removed net ADC3_4: U$18.2
- removed net ADC_TGS2611: C33.1, R57.2, R58.2
- removed net DAP: IC7.15
- removed net DGND: IC7.1
- removed net ENB_PWR_IF11: Q16.1, R79.2
- removed net ENB_PWR_IF12: Q17.1, R80.2
- removed net EN_IF11: Q16.3, R79.1, U$17.4
- removed net EN_IF12: Q17.3, R80.1, U$18.4
- removed net N$12 (its old number): C22.1, C4.1, R66.2
- removed net N$13 (its old number): C22.2
- removed net N$14: C4.2
- removed net N$16: IC2.5
- removed net N$17: R38.1
- removed net N$18: R34.2
- removed net N$26: R39.1, T3.1
- removed net N$27: C18.1
- removed net N$28: IC2.1, R34.1, R35.2
- removed net N$32: IC2.3, R36.2, R37.1
- removed net N$34: C19.1, R37.2
- removed net N$35: IC2.4, R36.1
- removed net N$36: C18.2, C19.2, R33.2, R39.2
- removed net N$46: IC8.17, TP18.TP
- removed net N$53: Q1.3, S$2.1
- removed net N$56: C34.1, IC3.4
- removed net PWM: R33.1
- removed net RS_NEG: R56.1, R57.1, S$2.2
- removed net RS_POS: C32.1, R60.2, R61.1, R62.1, S$2.3
- removed net TGS2611_HEAT_EN: Q1.1, R59.1
- removed net V-: IC2.2
- removed net VDD: IC7.6
- removed net VREF_TGS6211: R62.2
- removed net V_NEG: S$1.V_NEG
- removed net V_POS: S$1.V_POS
- new net 3AIN0: C18.1, IC2.5, R15.1
- new net 3AIN1: C19.1, IC2.6, R18.1
- new net N$7: IC2.2, TP21.TP
- net +5V/1: now also C4.1, C42.1, IC2.8, R67.1, R70.1, R71.1, R72.1, R73.1, R74.1, R75.1, R76.1, R77.1, R78.1; no longer Q16.2, Q17.2
- net 1AIN0: now also IC5.6; no longer IC5.4
- net 1AIN1: now also IC5.7; no longer IC5.5
- net 1AIN2: now also IC5.5; no longer IC5.7
- net 1AIN3: now also IC5.4; no longer IC5.6
- net 2AIN0: now also IC4.6; no longer IC4.4
- net 2AIN1: now also IC4.7; no longer IC4.5
- net 2AIN2: now also IC4.5; no longer IC4.7
- net 2AIN3: now also IC4.4; no longer IC4.6
- net 5V: no longer C35.1, C42.1, IC3.1, IC3.3, R60.1, S$2.4
- net 5V_CALM: no longer U$17.3, U$18.3
- net ADC3_1: now also R15.2
- net ADC3_2: now also R18.2
- net AGND: now also C18.2, C19.2, C4.2, IC2.3; no longer IC7.7, U$17.1, U$18.1
- net BTN1: now also R14.2
- net ENB_PWR_IF1: now also IC8.10; no longer IC8.4
- net ENB_PWR_IF10: now also IC8.4
- net ENB_PWR_IF2: now also IC8.11; no longer IC8.5
- net ENB_PWR_IF7: now also IC8.20; no longer IC8.10
- net ENB_PWR_IF8: now also IC8.19; no longer IC8.11
- net ENB_PWR_IF9: now also IC8.5
- net EN_IF1: no longer R67.1
- net EN_IF10: no longer R78.1
- net EN_IF2: no longer R70.1
- net EN_IF3: no longer R71.1
- net EN_IF4: no longer R72.1
- net EN_IF5: no longer R73.1
- net EN_IF6: no longer R74.1
- net EN_IF7: no longer R75.1
- net EN_IF8: no longer R76.1
- net EN_IF9: no longer R77.1
- net GND: no longer C32.2, C33.2, C34.2, C35.2, C36.2, IC3.2, Q1.2, R38.2, R56.2, R58.1, R59.2, T3.2
- net NRST: now also R14.1
- net SCL_5V: now also IC2.1, IC2.10; no longer U$17.6, U$18.6
- net SDA_5V: now also IC2.9; no longer U$17.5, U$18.5
Routing:
- net 5V_CALM: track 0.00 -> 283.1 mm, vias 0 -> 11
- net AGND: track 0.00 -> 229.5 mm, vias 0 -> 18
- net SCL_5V: track 0.00 -> 226.6 mm, vias 0 -> 9
- net SDA_5V: track 0.00 -> 183.0 mm, vias 0 -> 5
- net +5V/1: track 0.00 -> 93.3 mm, vias 0 -> 2
- net ENB_PWR_IF7: track 0.00 -> 82.3 mm, vias 0 -> 2
- net ENB_PWR_IF8: track 0.00 -> 80.4 mm, vias 0 -> 2
- net FAN_MCU: track 0.00 -> 61.0 mm, vias 0 -> 4
- net ENB_PWR_IF6: track 0.00 -> 41.5 mm
- net ENB_PWR_IF1: track 0.00 -> 38.7 mm
- net ENB_PWR_IF5: track 0.00 -> 35.9 mm
- net ENB_PWR_IF2: track 0.00 -> 32.1 mm
- net GND: track 597.8 -> 628.4 mm, vias 53 -> 57
- net EN_IF3: track 0.00 -> 28.1 mm, vias 0 -> 1
- net ADC2_3: track 0.00 -> 28.1 mm
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- added copper zone on layer 16, net 5V
Other:
- board text removed: "GND"

Commit message: layout done,
Parts:
- U$7: device FRA_eagle_lib:ETH_MODULE_OUTLINE -> FRA_eagle_lib:ETH_MODULE_OUTLINE_SMALL
- moved TP17 5.50 mm to (34.2, 55.7)
- moved TP16 5.30 mm to (32.7, 55.7)
- moved TP15 5.10 mm to (31.1, 55.7)
- moved TP14 4.06 mm to (29.6, 55.7)
- moved TP13 2.18 mm to (43.2, 59.1)
- moved TP6 0.31 mm to (91.2, 59.1)
- moved TP5 0.31 mm to (41.2, 33.3)
- renumbered SENSOR_D1 to S_D1, SENSOR_D2 to S_D2
Connections:
- removed net BTN2: U2.7
- new net N$14: IC2.4, SENSOR_D3.3
- new net N$16: IC2.7, SENSOR_D3.2
- net +5V/1: now also SENSOR_D3.4
- net AGND: now also SENSOR_D3.1
Routing:
- net +5V/1: track 93.3 -> 248.8 mm, vias 2 -> 20
- net AGND: track 229.5 -> 362.1 mm, vias 18 -> 53
- net SDA_5V: track 183.0 -> 290.0 mm, vias 5 -> 13
- net SCL_5V: track 226.6 -> 320.0 mm, vias 9 -> 13
- net GND: track 628.4 -> 578.6 mm, vias 57 -> 84
- net ADC3_1: track 0.00 -> 20.7 mm
- net N$14: track 0.00 -> 18.3 mm, vias 0 -> 2
- net N$16: track 0.00 -> 11.0 mm, vias 0 -> 1
- net ADC3_2: track 0.00 -> 5.90 mm
- net N$9: track 1.76 -> 6.09 mm
- net N$12: track 1.79 -> 4.95 mm
- net N$10: track 2.40 -> 5.51 mm
- net N$13: track 2.48 -> 4.57 mm
- net 5V_CALM_LDO: track 5.97 -> 7.72 mm
- net ENB_PWR_IF7: track 82.3 -> 83.9 mm
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- added copper zone on layer 1, net +5V/1
- added copper zone on layer 16, net +5V/1
- added copper zone on layer 1, net AGND
- added copper zone on layer 16, net AGND
Other:
- board size 100 x 100 mm -> 100.3 x 100 mm
- board text added: "*"
- board text added: "+"
- board text added: "07/2019"
- board text removed: "06/2019"

Commit message: updates
Parts:
- removed FID3: FIDUCIAL"", microbuilder:FIDUCIAL_1MM
- added C20: 10u, resistor:C0603K
- added C22: 100n, resistor:C0603K
- added IC3: P82B715DR, SamacSys_Parts:SOIC127P600X175-8N
- added R33, R34: 330, resistor:R0603
- R21: value 1M -> 100k
- R3: value 470 -> 100
- renumbered SENSOR_D3 to J9
Connections:
- new net SCL_BUFF: IC3.7, R34.2, U$10.6, U$11.6, U$12.6, U$13.6, U$14.6, U$15.6, U$16.6, U$3.6, U$8.6, U$9.6
- new net SDA_BUFF: IC3.2, R33.2, U$10.5, U$11.5, U$12.5, U$13.5, U$14.5, U$15.5, U$16.5, U$3.5, U$8.5, U$9.5
- net +5V/1: now also C20.1, C22.1, IC3.8, R33.1, R34.1
- net AGND: now also C20.2, C22.2, IC3.4
- net SCL_5V: now also IC3.6; no longer U$10.6, U$11.6, U$12.6, U$13.6, U$14.6, U$15.6, U$16.6, U$3.6, U$8.6, U$9.6
- net SDA_5V: now also IC3.3; no longer U$10.5, U$11.5, U$12.5, U$13.5, U$14.5, U$15.5, U$16.5, U$3.5, U$8.5, U$9.5
Routing:
- net SCL_BUFF: track 0.00 -> 225.8 mm, vias 0 -> 6
- net SDA_BUFF: track 0.00 -> 205.6 mm, vias 0 -> 8
- net SCL_5V: track 320.0 -> 115.0 mm, vias 13 -> 8
- net SDA_5V: track 290.0 -> 114.0 mm, vias 13 -> 8
- net +5V/1: track 248.8 -> 276.6 mm, vias 20 -> 22
- net VIN: track 19.2 -> 22.9 mm
- net AGND: track 362.1 -> 363.9 mm, vias 53 -> 52
- net ENB_PWR_IF1: track 38.7 -> 38.2 mm
Other:
- board text added: "+7-12V"
- board text added: "A1.0"
- board text added: "A1.1"
- board text added: "A1.2"
- board text added: "A1.3"
- board text added: "A2.0"
- board text added: "A2.1"
- board text added: "A2.2"
- board text added: "A2.3"
- board text added: "A3.0,A3.3"
- board text added: "A3.1"
- board text added: "A3.2"
- board text added: "ALLPCB marking"
- board text added: "GND"
- board text added: "J.Repcik"
- board text removed: "01-16"
- board text removed: "01-20"
- board text removed: "Juraj Repcik"
- board text removed: "LAYER-STACK"
