File: 2-Electrical/0 - Development Drawings/2-SensorBoard/5-CAD_Project/FRA_daughter_v1.brd (EAGLE design)
At the start: 75 x 40 mm, 64 parts, among them IC1 LMV611, IC3 LMV796MF_NOPB, IC4 LMP91000SD_NOPB, IC5 REF3125AQDBZRQ1, IC6 MCP6541T-I_OT, J1 INSERT_MM5_06691.5MM, J10 2wire, J2 TGS3, J3 TGS2, J4 TGS1, J5 TGS4, J6 INSERT_MM5_06691.5MM, J7 INSERT_MM5_06691.5MM, J8 INSERT_MM5_06691.5MM, J9 INSERT_MM5_06691.5MM, Q1 PMBFJ177,215, Q3 Si2300DS, X1 3-ELECTRODE-GAS-SENSORINS

Commit message: BOM updates, labview
Parts:
- added C12, C4, C9: 100n, resistor:C0603K
- flipped U$1 to the bottom
Connections:
- net 5V_CALM: now also C12.2, C4.2
- net AGND: now also C12.1, C4.1, C9.2
- net VOUT: now also C9.1
Routing:
- net VOUT: track 15.5 -> 30.6 mm, vias 0 -> 3
- net GND: track 169.2 -> 176.0 mm, vias 3 -> 9
- net SCL: track 28.4 -> 23.1 mm
- net 5V_CALM: track 109.5 -> 114.3 mm, vias 6 -> 7
- net SDA: track 30.2 -> 30.5 mm, vias 1 -> 3
- net AGND: vias 7 -> 25
Other:
- board text added: "1"
- board text added: "2"
- board text added: "3"
- board text added: "4"
- board text added: "BOT"
- board text added: "MG-812 TGS4161"
- board text added: "Sensor PCB v1 J.Repcik 7/2019"
- board text added: "TGS2611 TGS2612 TGS2620"
- board text added: "TGS5042"
- board text added: "TOP"
- board text added: "U$1 con. BOTTOM assembly"
