File: 2-Electrical/0 - Development Drawings/2-SensorBoard/5-CAD_Project/FRA_daughter_v1.sch (EAGLE design)
At the start: 64 parts, among them IC1 LMV611, IC3 LMV796MF_NOPB, IC4 LMP91000SD_NOPB, IC5 REF3125AQDBZRQ1, IC6 MCP6541T-I_OT, J1 INSERT_MM5_06691.5MM, J10 2wire, J2 TGS3, J3 TGS2, J4 TGS1, J5 TGS4, J6 INSERT_MM5_06691.5MM, J7 INSERT_MM5_06691.5MM, J8 INSERT_MM5_06691.5MM, J9 INSERT_MM5_06691.5MM, Q1 PMBFJ177,215, Q3 Si2300DS, X1 3-ELECTRODE-GAS-SENSORINS

Commit message: BOM updates, labview
Parts:
- added C12, C4, C9: 100n, resistor:C-EUC0603K
Connections:
- net 5V_CALM: now also C12.2, C4.2
- net AGND: now also C12.1, C4.1, C9.2
- net VOUT: now also C9.1
