File: 2-Electrical/0 - Development Drawings/3-SensorTGS2xxx_board/5-CADProject/FRA_Sensor_TGS2xxx.brd (EAGLE design)
At the start: 20 x 30 mm, 29 parts, among them IC3 LMV796MF_NOPB, IC6 MCP6541T-I_OT, J1 CONN_03X2_WE_61200621621, Q3 Si2300DS, U2 FIGARO_SR-7

Commit message: amonia sensor tuning
Parts:
- C13: value 100n -> 1n
- J1: value CONN_03X2_WE_61200621621 -> CONN_03X2
