File: 2-Electrical/0 - Development Drawings/5-MHM01_board/5-CAD_Project/V1/MHM01.brd (EAGLE design)
At the start: 33 x 40 mm, 33 parts, among them Q1 Si2300DS, U2 FIGARO_SR-7, X1 TB001-500-02BE, X2 TB001-500-02BE, X3 TB001-500-02BE

Commit message: BOM updates
Parts:
- LED2: value (none) -> Red
- R12: value (none) -> 100
Changed lines of the file:
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@@
 <attribute name="NAME" x="25.656" y="29.718" size="0.8128" layer="25" rot="R180" align="center"/>
 <attribute name="VALUE" x="26.663" y="29.522" size="1.27" layer="27" rot="R180" align="center"/>
+<attribute name="PARTNO" value="AP2202K-ADJTRG1" x="26.663" y="32.062" size="1.778" layer="27" rot="R180" display="off"/>
 </element>
 <element name="R2" library="resistor" package="R0603" value="10k" x="26.147" y="37.532" smashed="yes">
 <attribute name="NAME" x="25.258" y="38.294" size="0.8128" layer="25"/>
 <attribute name="VALUE" x="25.512" y="35.627" size="1.27" layer="27"/>
+<attribute name="PARTNO" value="CRCW060310K0FKEA" x="26.147" y="37.532" size="1.778" layer="27" display="off"/>
 </element>
 <element name="R3" library="resistor" package="R0603" value="3k" x="22.591" y="36.525" smashed="yes" rot="R90">
 <attribute name="NAME" x="21.659" y="35.264" size="0.8128" layer="25" rot="R90"/>
 <attribute name="VALUE" x="24.496" y="35.89" size="1.27" layer="27" rot="R90"/>
+<attribute name="PARTNO" value="ERA-3AEB302V" x="22.591" y="36.525" size="1.778" layer="27" rot="R90" display="off"/>
 </element>
 <element name="C3" library="resistor" package="C0603K" value="1u" x="30.6" y="32.062" smashed="yes" rot="R90">
 <attribute name="NAME" x="29.942" y="31.335" size="0.8128" layer="25" rot="R90"/>
 <attribute name="VALUE" x="32.25" y="31.262" size="1.016" layer="27" rot="R90"/>
+<attribute name="PARTNO" value="GRM188R71C105KE15D" x="30.6" y="32.062" size="1.778" layer="27" rot="R90" display="off"/>
 </element>
 <element name="C5" library="resistor" package="C0603K" value="10u" x="20.231" y="32.07" smashed="yes" rot="R90">
 <attribute name="NAME" x="19.29" y="31.397" size="0.8128" layer="25" rot="R90"/>
 <attribute name="VALUE" x="21.881" y="31.27" size="1.016" layer="27" rot="R90"/>
+<attribute name="PARTNO" value="GRM188R61A106KE69J" x="20.231" y="32.07" size="1.778" layer="27" rot="R90" display="off"/>
 </element>
 <element name="C7" library="resistor" package="C0603K" value="100n" x="21.182" y="29.125" smashed="yes">
 <attribute name="NAME" x="20.583" y="29.886" size="0.8128" layer="25"/>
 <attribute name="VALUE" x="20.382" y="27.475" size="1.016" layer="27"/>
+<attribute name="PARTNO" value="CC0603KRX7R8BB104" x="21.182" y="29.125" size="1.778" layer="27" display="off"/>
 </element>
 <element name="U$1" library="FRA_eagle_lib" package="WE_61200621621" value="CONN_03X2_WE_61200621621" x="26.942" y="20.816" smashed="yes">
 <attribute name="NAME" x="22.878" y="27.801" size="0.8128" layer="25" font="vector" ratio="20"/>
 <attribute name="VALUE" x="22.878" y="13.45" size="0.6096" layer="27" font="vector" ratio="20"/>
+<attribute name="PARTNO" value="61200621621" x="26.942" y="20.816" size="1.778" layer="27" display="off"/>
 </element>
 <element name="FID1" library="microbuilder" package="FIDUCIAL_1MM" value="FIDUCIAL&quot;&quot;" x="2.845" y="32.495" smashed="yes"/>
@@
 </element>
 <element name="U2" library="FRA_eagle_lib" package="FIGARO-SR7" value="FIGARO_SR-7" x="12.06" y="33.615" smashed="yes" rot="R180">
-<attribute name="PARTNO" value="installed_by_customer" x="12.06" y="33.615" size="1.778" layer="27" rot="R180" display="off"/>
+<attribute name="PARTNO" value="SR-7" x="12.06" y="33.615" size="1.778" layer="27" rot="R180" display="off"/>
 <attribute name="NAME" x="9.475" y="28.85" size="0.8128" layer="25" rot="R180"/>
 <attribute name="VALUE" x="9.52" y="38.695" size="1.27" layer="27" rot="R180"/>
@@
 <attribute name="NAME" x="22.3188" y="1.7962" size="1.27" layer="25" ratio="10"/>
 </element>
-<element name="LED2" library="adafruit" package="CHIPLED_1206" value="" x="20.43" y="25.11" smashed="yes" rot="R180">
+<element name="LED2" library="adafruit" package="CHIPLED_1206" value="Red" x="20.43" y="25.11" smashed="yes" rot="R180">
 <attribute name="NAME" x="18.73" y="26.335" size="0.8128" layer="25" rot="R270"/>
 <attribute name="VALUE" x="17.89" y="26.38" size="1.27" layer="27" rot="R270"/>
+<attribute name="PARTNO" value="BR1101W-TR" x="20.43" y="25.11" size="1.778" layer="27" rot="R180" display="off"/>
 </element>
 <element name="FB1" library="microbuilder" package="0603" value="" x="29.205" y="28.89" smashed="yes" rot="R180">
@@
 <attribute name="NAME" x="25.195" y="35.6" size="0.8128" layer="25"/>
 <attribute name="VALUE" x="25.51" y="33.195" size="1.27" layer="27"/>
+<attribute name="PARTNO" value="CRCW060310K0FKEA" x="26.145" y="35.1" size="1.778" layer="27" display="off"/>
 </element>
 <element name="R9" library="resistor" package="R0603" value="220" x="22.59" y="32.04" smashed="yes" rot="R90">
 <attribute name="NAME" x="21.865" y="31.585" size="0.8128" layer="25" rot="R90"/>
 <attribute name="VALUE" x="24.495" y="31.405" size="1.27" layer="27" rot="R90"/>
+<attribute name="PARTNO" value="CRCW0603220RFKEA" x="22.59" y="32.04" size="1.778" layer="27" rot="R90" display="off"/>
 </element>
-<element name="R12" library="pot" package="RJ9W" value="" x="6.03" y="24.255" smashed="yes" rot="R180">
+<element name="R12" library="pot" package="RJ9W" value="100" x="6.03" y="24.255" smashed="yes" rot="R180">
 <attribute name="NAME" x="10.602" y="21.588" size="0.8128" layer="25" ratio="10" rot="R180"/>
 <attribute name="VALUE" x="10.602" y="28.319" size="1.27" layer="27" ratio="10" rot="R180"/>
+<attribute name="PARTNO" value="3296X-1-101LF" x="6.03" y="24.255" size="1.778" layer="27" rot="R180" display="off"/>
 </element>
 <element name="R19" library="rcl" package="R1206" value="DNI" x="4.59" y="28.17" smashed="yes">
@@
 <attribute name="NAME" x="4.465" y="16.21" size="0.8128" layer="25" rot="R270"/>
 <attribute name="VALUE" x="0.655" y="16.21" size="1.27" layer="27" rot="R270"/>
+<attribute name="PARTNO" value="CRCW120675R0FKEA" x="3.195" y="14.94" size="1.778" layer="27" rot="R270" display="off"/>
 </element>
 <element name="R21" library="rcl" package="R1206" value="75" x="7.2" y="15.075" smashed="yes" rot="R90">
 <attribute name="NAME" x="9.17" y="14.435" size="0.8128" layer="25" rot="R90"/>
 <attribute name="VALUE" x="9.74" y="13.805" size="1.27" layer="27" rot="R90"/>
+<attribute name="PARTNO" value="CRCW120675R0FKEA" x="7.2" y="15.075" size="1.778" layer="27" rot="R90" display="off"/>
 </element>
 <element name="R7" library="rcl" package="R1206" value="75" x="11.205" y="14.985" smashed="yes" rot="R270">
 <attribute name="NAME" x="12.43" y="15.715" size="0.8128" layer="25" rot="R270"/>
 <attribute name="VALUE" x="8.665" y="16.255" size="1.27" layer="27" rot="R270"/>
+<attribute name="PARTNO" value="CRCW120675R0FKEA" x="11.205" y="14.985" size="1.778" layer="27" rot="R270" display="off"/>
 </element>
 <element name="R22" library="rcl" package="R1206" value="10K" x="14.31" y="15.03" smashed="yes" rot="R90">
 <attribute name="NAME" x="16.19" y="14.21" size="0.8128" layer="25" rot="R90"/>
 <attribute name="VALUE" x="16.85" y="13.76" size="1.27" layer="27" rot="R90"/>
+<attribute name="PARTNO" value="CRCW120610K0FKEA" x="14.31" y="15.03" size="1.778" layer="27" rot="R90" display="off"/>
 </element>
 <element name="Q1" library="adafruit" package="SOT23" value="Si2300DS" x="14.985" y="21.285" smashed="yes">
@@
 <attribute name="NAME" x="19.9" y="15.38" size="0.8128" layer="25" rot="R180"/>
 <attribute name="VALUE" x="19.9" y="19.19" size="1.27" layer="27" rot="R180"/>
+<attribute name="PARTNO" value="JMF316AB7106KLHT" x="18.63" y="16.65" size="1.778" layer="27" rot="R180" display="off"/>
 </element>
 <element name="C2" library="rcl" package="C1206" value="10u" x="18.585" y="13.14" smashed="yes" rot="R180">
 <attribute name="NAME" x="19.855" y="11.87" size="0.8128" layer="25" rot="R180"/>
 <attribute name="VALUE" x="19.855" y="15.68" size="1.27" layer="27" rot="R180"/>
+<attribute name="PARTNO" value="JMF316AB7106KLHT" x="18.585" y="13.14" size="1.778" layer="27" rot="R180" display="off"/>
 </element>
 <element name="R1" library="rcl" package="R1206" value="75" x="17.685" y="24.93" smashed="yes" rot="R270">
 <attribute name="NAME" x="15.715" y="25.885" size="0.8128" layer="25" rot="R270"/>
 <attribute name="VALUE" x="15.145" y="26.2" size="1.27" layer="27" rot="R270"/>
+<attribute name="PARTNO" value="CRCW120675R0FKEA" x="17.685" y="24.93" size="1.778" layer="27" rot="R270" display="off"/>
 </element>
 <element name="R4" library="rcl" package="R1206" value="0" x="19.035" y="38.25" smashed="yes" rot="R180">
 <attribute name="NAME" x="20.305" y="36.98" size="0.8128" layer="25" rot="R180"/>
 <attribute name="VALUE" x="20.305" y="40.79" size="1.27" layer="27" rot="R180"/>
+<attribute name="PARTNO" value="CRCW12060000Z0EA" x="19.035" y="38.25" size="1.778" layer="27" rot="R180" display="off"/>
 </element>
 </elements>
