File: 2-Electrical/0 - Development Drawings/5-MHM01_board/5-CAD_Project/V1/MHM01.sch (EAGLE design)
At the start: 33 parts, among them Q1 Si2300DS, U2 FIGARO_SR-7, X1 TB001-500-02BE, X2 TB001-500-02BE, X3 TB001-500-02BE

Commit message: BOM updates
Parts:
- C1, C2: PARTNO (none) -> JMF316AB7106KLHT
- C3: PARTNO (none) -> GRM188R71C105KE15D
- C5: PARTNO (none) -> GRM188R61A106KE69J
- C7: PARTNO (none) -> CC0603KRX7R8BB104
- LED2: value (none) -> Red; PARTNO (none) -> BR1101W-TR
- PS1: PARTNO (none) -> AP2202K-ADJTRG1
- R1, R20, R21, R7: PARTNO (none) -> CRCW120675R0FKEA
- R12: value (none) -> 100; PARTNO (none) -> 3296X-1-101LF
- R2, R8: PARTNO (none) -> CRCW060310K0FKEA
- R22: PARTNO (none) -> CRCW120610K0FKEA
- R3: PARTNO (none) -> ERA-3AEB302V
- R4: PARTNO (none) -> CRCW12060000Z0EA
- R9: PARTNO (none) -> CRCW0603220RFKEA
- U$1: PARTNO (none) -> 61200621621
- U2: PARTNO installed_by_customer -> SR-7
Other:
- note added: "MHM01 fists to ST-7 as follows: SR7 pin MHM01 pin Function 1 2 sensor - 2 NC 3 NC 4 1 sensor+"
- note added: "RA"
- note added: "RB"
- note added: "VOUT=1.25* (1+RB/RA)"
- note removed: "MHM01 fists to ST-7 as follows: ST7 pin MHM01 pin Function 1 2 sensor - 2 NC 3 NC 4 1 sensor+"
- note removed: "VOUT=1.25* (1+R2/R3)"
