File: 2-Electrical/0 - Development Drawings/6-Breakout_10U/5 - CAD project/FRA_junctionB_v1.brd (EAGLE design)
At the start: 100 x 55 mm, 24 parts, among them U1 SSW-103-01-F-D, U10 SSW-103-01-F-D, U11 TB003V-500-P05BE, U12 TB003V-500-P10BE, U13 TB003V-500-P05BE, U14 TB003V-500-P10BE, U2 SSW-103-01-F-D, U3 SSW-103-01-F-D, U4 SSW-103-01-F-D, U5 SSW-103-01-F-D, U6 SSW-103-01-F-D, U7 SSW-103-01-F-D, U8 SSW-103-01-F-D, U9 SSW-103-01-F-D

Commit message: silkscreen edits on breakout boards
Other:
- board text added: "5V --- A1.2 --- GND --- 5V --- A1.1 --- GND --- 5V A3.1 --- GND --- 5V --- A2.2 --- GND --- 5V --- A2.1 --- GND"
- board text added: "5V --- A1.3 --- GND --- 5V --- A1.0 --- GND --- 5V A3.2 --- GND --- 5V --- A2.3 --- GND --- 5V --- A2.0 --- GND"
- board text added: "J. Repcik 12/2020"
- board text removed: "5V --- A1.1 --- GND --- 5V --- A1.3 --- GND --- 5V A3.1 --- GND --- 5V --- A2.1 --- GND --- 5V --- A2.3 --- GND"
- board text removed: "5V --- A1.2 --- GND --- 5V --- A1.4 --- GND --- 5V A3.2 --- GND --- 5V --- A2.2 --- GND --- 5V --- A2.4 --- GND"
- board text removed: "J. Repcik 03/2020"
Changed lines of the file:
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@@
 <?xml version="1.0" encoding="utf-8"?>
 <!DOCTYPE eagle SYSTEM "eagle.dtd">
-<eagle version="9.5.2">
+<eagle version="9.6.2">
 <drawing>
 <settings>
-<setting alwaysvectorfont="yes"/>
+<setting alwaysvectorfont="no"/>
 <setting keepoldvectorfont="yes"/>
 <setting verticaltext="up"/>
@@
 <layer number="24" name="bOrigins" color="15" fill="1" visible="no" active="yes"/>
 <layer number="25" name="tNames" color="58" fill="1" visible="yes" active="yes"/>
-<layer number="26" name="bNames" color="7" fill="1" visible="no" active="yes"/>
+<layer number="26" name="bNames" color="7" fill="1" visible="yes" active="yes"/>
 <layer number="27" name="tValues" color="7" fill="1" visible="no" active="yes"/>
 <layer number="28" name="bValues" color="7" fill="1" visible="no" active="yes"/>
@@
 <text x="22.54" y="27" size="1.5" layer="51" font="vector" ratio="15">Electronics design solutions s.r.o.</text>
 <text x="22.54" y="29" size="2" layer="51" font="vector" ratio="15">FRA Sensor unit junction board</text>
-<text x="22.54" y="25" size="1.5" layer="51" font="vector" ratio="15">J. Repcik 03/2020</text>
+<text x="22.54" y="25" size="1.5" layer="51" font="vector" ratio="15">J. Repcik 12/2020</text>
 <dimension x1="100" y1="55" x2="0" y2="55" x3="50" y3="59" textsize="1.778" layer="47"/>
 <dimension x1="100" y1="0" x2="100" y2="55" x3="106" y3="27.5" textsize="1.778" layer="47"/>
@@
 <text x="85.871" y="6.284" size="1.66" layer="51" font="vector" ratio="15" rot="R90" align="bottom-right">5V
 ---
-A1.2
+A1.3
 ---
 GND
@@
 5V
 ---
-A1.4
+A1.0
 ---
 GND
@@
 5V
 ---
-A2.2
+A2.3
 ---
 GND
@@
 5V
 ---
-A2.4
+A2.0
 ---
 GND</text>
 <text x="85.871" y="54.925" size="1.66" layer="51" font="vector" ratio="15" rot="R90" align="bottom-right">5V
 ---
+A1.2
+---
+GND
+---
+5V
+---
 A1.1
----
-GND
----
-5V
----
-A1.3
 ---
 GND
@@
 5V
 ---
+A2.2
+---
+GND
+---
+5V
+---
 A2.1
 ---
-GND
----
-5V
----
-A2.3
----
 GND</text>
