File: 2-Electrical/0 - Development Drawings/7-Breakout_6U/5 - CAD project/FRA_breakout6U_v1.brd (EAGLE design)
At the start: 51 x 67 mm, 14 parts, among them U10 SSW-103-01-F-D, U12 TB003V-500-P10BE, U14 TB003V-500-P10BE, U5 SSW-103-01-F-D, U6 SSW-103-01-F-D, U7 SSW-103-01-F-D, U8 SSW-103-01-F-D, U9 SSW-103-01-F-D

Commit message: silkscreen edits on breakout boards
Other:
- board text added: "--- GND --- 5V --- A3.1 --- GND --- 5V --- A2.2 --- GND --- 5V --- A2.1 --- GND"
- board text added: "--- GND --- 5V --- A3.2 --- GND --- 5V --- A2.3 --- GND --- 5V --- A2.0 --- GND"
- board text added: "J. Repcik 12/2020"
- board text removed: "--- GND --- 5V --- A3.1 --- GND --- 5V --- A2.1 --- GND --- 5V --- A2.3 --- GND"
- board text removed: "--- GND --- 5V A3.2 --- GND --- 5V --- A2.2 --- GND --- 5V --- A2.4 --- GND"
- board text removed: "J. Repcik 03/2020"
Changed lines of the file:
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@@
 <?xml version="1.0" encoding="utf-8"?>
 <!DOCTYPE eagle SYSTEM "eagle.dtd">
-<eagle version="9.5.2">
+<eagle version="9.6.2">
 <drawing>
 <settings>
@@
 <text x="7.54" y="32" size="1.5" layer="51" font="vector" ratio="15">Electronics design solutions s.r.o.</text>
 <text x="7.54" y="34" size="2" layer="51" font="vector" ratio="15">Breakout 6U</text>
-<text x="7.54" y="30" size="1.5" layer="51" font="vector" ratio="15">J. Repcik 03/2020</text>
+<text x="7.54" y="30" size="1.5" layer="51" font="vector" ratio="15">J. Repcik 12/2020</text>
 <wire x1="19.001" y1="27.86" x2="18.493" y2="27.86" width="0.3048" layer="51"/>
 <wire x1="18.493" y1="27.86" x2="18.366" y2="27.733" width="0.3048" layer="51"/>
@@
 ---
 5V
+---
 A3.2
 ---
@@
 5V
 ---
-A2.2
+A2.3
 ---
 GND
@@
 5V
 ---
-A2.4
+A2.0
 ---
 GND</text>
@@
 5V
 ---
+A2.2
+---
+GND
+---
+5V
+---
 A2.1
 ---
-GND
----
-5V
----
-A2.3
----
 GND</text>
