File: 2-Electrical/0 - Development Drawings/8-Universal_Bulkhead/5 - CAD project/FRA_bulkhead_v2.brd (EAGLE design)
At the start: 112 x 83 mm, 43 parts, among them J9 4pin, U1 TB003V-500-P05BERIGHTANGLE-NO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, U2 TB003V-500-P10BERIGHTANGLE-NO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, U22 TB003V-500-P05BERIGHTANGLE-NO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, U23 TB003V-500-P10BERIGHTANGLE-NO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, U3 TB003V-500-P05BERIGHTANGLE-NO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, X1 TB001-500-02BE

Commit message: silkscreen edits on breakout boards
Other:
- board text added: "+5V A1.2 GND +5V A1.1 GND +5V A3.1 GND +5V A2.2 GND +5V A2.1 GND"
- board text added: "+5V A1.3 GND +5V A1.0 GND +5V A3.2 GND +5V A2.3 GND +5V A2.0 GND"
- board text added: "J.Repcik / 12/2020"
- board text removed: "+5V A1.1 GND +5V A1.3 GND +5V A3.1 GND +5V A2.1 GND +5V A2.3 GND"
- board text removed: "+5V A1.2 GND +5V A1.4 GND +5V A3.2 GND +5V A2.2 GND +5V A2.4 GND"
- board text removed: "J.Repcik / 03/2020"
Changed lines of the file:
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@@
 <?xml version="1.0" encoding="utf-8"?>
 <!DOCTYPE eagle SYSTEM "eagle.dtd">
-<eagle version="9.5.2">
+<eagle version="9.6.2">
 <drawing>
 <settings>
@@
 <layer number="14" name="Route14" color="1" fill="6" visible="no" active="no"/>
 <layer number="15" name="Route15" color="4" fill="6" visible="no" active="no"/>
-<layer number="16" name="Bottom" color="1" fill="1" visible="no" active="yes"/>
+<layer number="16" name="Bottom" color="1" fill="1" visible="yes" active="yes"/>
 <layer number="17" name="Pads" color="2" fill="1" visible="yes" active="yes"/>
 <layer number="18" name="Vias" color="2" fill="1" visible="yes" active="yes"/>
@@
 <text x="25.566865625" y="103.68180625" size="1.5" layer="51" font="vector" ratio="15" rot="R90">GND +5V</text>
 <text x="124.82" y="99.436" size="1.25" layer="51" font="vector" ratio="15" rot="R270">GND A3.3 A3.0 +5V +5V</text>
-<text x="48.164" y="120.22" size="1.3" layer="51" font="vector" ratio="15">+5V A1.1 GND +5V A1.3 GND +5V A3.1 GND +5V A2.1 GND +5V A2.3 GND</text>
-<text x="48.264" y="51.02" size="1.3" layer="51" font="vector" ratio="15">+5V A1.2 GND +5V A1.4 GND +5V A3.2 GND +5V A2.2 GND +5V A2.4 GND</text>
+<text x="48.164" y="120.22" size="1.3" layer="51" font="vector" ratio="15">+5V A1.2 GND +5V A1.1 GND +5V A3.1 GND +5V A2.2 GND +5V A2.1 GND</text>
+<text x="48.264" y="51.02" size="1.3" layer="51" font="vector" ratio="15">+5V A1.3 GND +5V A1.0 GND +5V A3.2 GND +5V A2.3 GND +5V A2.0 GND</text>
 <text x="89.636" y="47.976" size="1" layer="51" font="vector" ratio="15">Electronics design solutions s.r.o.</text>
-<text x="89.536" y="46.276" size="1" layer="51" font="vector" ratio="15">J.Repcik / 03/2020</text>
+<text x="89.536" y="46.276" size="1" layer="51" font="vector" ratio="15">J.Repcik / 12/2020</text>
 <wire x1="42.901" y1="95.86" x2="42.393" y2="95.86" width="0.3048" layer="51"/>
 <wire x1="42.393" y1="95.86" x2="42.266" y2="95.733" width="0.3048" layer="51"/>
